Commit message: launchfiles update

File: mrvk_description/urdf/mrvk.urdf.xacro (robot description, xacro)
@@ -46,5 +46,5 @@
    </link>
   <joint name="stabilizer_to_imu" type="fixed">
-    <origin xyz="-0.1 0.1 -0.01"/>
+    <origin xyz="0.0 0.0 0.0"/>
     <parent link="base_stabilized"/>
     <child link="imu"/>
